Commit message: x

File: src/description/urdf/mobile_base.xacro (robot description, xacro)
@@ -74,6 +74,6 @@
         <parent link="base_link" />
         <child link="right_wheel_link" />
-        <!-- 0.001 is margin in reall world -->
-        <origin xyz="0 ${-(base_width + wheel_length + 0.001) / 2.0} -${wheel_support_length }" rpy="0 0 0" />
+        <!-- 0.01 is margin in real world -->
+        <origin xyz="0 ${-(base_width + wheel_length + 0.01) / 2.0} -${wheel_support_length }" rpy="0 0 0" />
         <axis xyz="0 1 0" />
     </joint>
@@ -81,6 +81,6 @@
         <parent link="base_link" />
         <child link="left_wheel_link" />
-        <!-- 0.001 is margin in reall world -->
-        <origin xyz="0 ${(base_width + wheel_length + 0.001) / 2.0} -${wheel_support_length}" rpy="0 0 0" />
+        <!-- 0.01 is margin in real world -->
+        <origin xyz="0 ${(base_width + wheel_length + 0.01) / 2.0} -${wheel_support_length}" rpy="0 0 0" />
         <axis xyz="0 1 0" />
     </joint>

File: src/description/urdf/mobile_base_gazebo.xacro (robot description, xacro)
@@ -9,5 +9,5 @@
             <left_joint>base_left_wheel_joint</left_joint>
             <right_joint>base_right_wheel_joint</right_joint>
-            <wheel_separation>0.36</wheel_separation>
+            <wheel_separation>0.335</wheel_separation>
             <wheel_radius>0.034</wheel_radius>
             <frame_id>odom</frame_id>

File: src/description/urdf/urdf_control_gz.xacro (robot description, xacro)
@@ -3,4 +3,4 @@
     <xacro:include filename="common_properties.xacro" />
     <xacro:include filename="mobile_base.xacro" />
-    <xacro:include filename="mobile_base.ros2_control_mock.xacro" />
+    <xacro:include filename="mobile_base.ros2_control_gz.xacro" />
 </robot>

Commit message: change 0.034 to 0.038 wheel

File: src/description/urdf/mobile_base.xacro (robot description, xacro)
@@ -6,5 +6,5 @@
     <xacro:property name="base_x_offset" value="0.075" />
     <xacro:property name="base_ground" value="0.055" />
-    <xacro:property name="wheel_radius" value="0.034" />
+    <xacro:property name="wheel_radius" value="0.038" />
     <xacro:property name="wheel_length" value="0.025" />
     <xacro:property name="wheel_support_length" value="${base_ground - wheel_radius}" />

File: src/description/urdf/mobile_base_gazebo.xacro (robot description, xacro)
@@ -10,5 +10,5 @@
             <right_joint>base_right_wheel_joint</right_joint>
             <wheel_separation>0.335</wheel_separation>
-            <wheel_radius>0.034</wheel_radius>
+            <wheel_radius>0.038</wheel_radius>
             <frame_id>odom</frame_id>
             <child_frame_id>base_footprint</child_frame_id>

Commit message: change 0.335 to 0.345 wheel separation

File: src/description/urdf/mobile_base.xacro (robot description, xacro)
@@ -75,5 +75,5 @@
         <child link="right_wheel_link" />
         <!-- 0.01 is margin in real world -->
-        <origin xyz="0 ${-(base_width + wheel_length + 0.01) / 2.0} -${wheel_support_length }" rpy="0 0 0" />
+        <origin xyz="0 ${-(base_width + wheel_length + 0.02) / 2.0} -${wheel_support_length }" rpy="0 0 0" />
         <axis xyz="0 1 0" />
     </joint>
@@ -82,5 +82,5 @@
         <child link="left_wheel_link" />
         <!-- 0.01 is margin in real world -->
-        <origin xyz="0 ${(base_width + wheel_length + 0.01) / 2.0} -${wheel_support_length}" rpy="0 0 0" />
+        <origin xyz="0 ${(base_width + wheel_length + 0.02) / 2.0} -${wheel_support_length}" rpy="0 0 0" />
         <axis xyz="0 1 0" />
     </joint>

File: src/description/urdf/mobile_base_gazebo.xacro (robot description, xacro)
@@ -9,5 +9,5 @@
             <left_joint>base_left_wheel_joint</left_joint>
             <right_joint>base_right_wheel_joint</right_joint>
-            <wheel_separation>0.335</wheel_separation>
+            <wheel_separation>0.345</wheel_separation>
             <wheel_radius>0.038</wheel_radius>
             <frame_id>odom</frame_id>
